File: schematics/schematics.kicad_sch (KiCad schematic)
At the start: 13 parts, among them J1 VRef, J2 Vmeas, U1 MCP602, U2 MCP602

Commit message: updated
Parts:
- removed A1: Arduino_Nano_Every, Module:Arduino_Nano, symbol MCU_Module:Arduino_Nano_Every
- added C1, C2: C, Capacitor_THT:CP_Axial_L10.0mm_D4.5mm_P15.00mm_Horizontal, symbol Device:C
- added J3: Conn_02x03_Odd_Even, Connector_PinHeader_2.54mm:PinHeader_2x03_P2.54mm_Vertical, symbol Connector_Generic:Conn_02x03_Odd_Even
- added J5: Conn_01x02_Pin, Connector_PinHeader_2.54mm:PinHeader_1x02_P2.54mm_Vertical, symbol Connector:Conn_01x02_Pin
- added J6: Conn_01x04_Pin, Connector_PinHeader_2.54mm:PinHeader_1x04_P2.54mm_Vertical, symbol Connector:Conn_01x04_Pin
- added R11, R6: 3k, Resistor_THT:R_Axial_DIN0207_L6.3mm_D2.5mm_P10.16mm_Horizontal, symbol Device:R
- added R2: 12k, Resistor_THT:R_Axial_DIN0207_L6.3mm_D2.5mm_P10.16mm_Horizontal, symbol Device:R
- added R5: 10k, Resistor_THT:R_Axial_DIN0207_L6.3mm_D2.5mm_P10.16mm_Horizontal, symbol Device:R
- added U3: ATmega328-P, Package_DIP:DIP-28_W7.62mm, symbol MCU_Microchip_ATmega:ATmega328-P
- J1, J2: footprint (none) -> Connector_Pin:Pin_D1.0mm_L10.0mm
- R1, R3, R4, R7, R8: value R -> 1k; footprint (none) -> Resistor_THT:R_Axial_DIN0207_L6.3mm_D2.5mm_P10.16mm_Horizontal
- R10, R9: value R -> 10k; footprint (none) -> Resistor_THT:R_Axial_DIN0207_L6.3mm_D2.5mm_P10.16mm_Horizontal
- Rm1: renamed from Rm; footprint (none) -> Resistor_THT:R_Axial_DIN0204_L3.6mm_D1.6mm_P2.54mm_Vertical
- U1, U2: footprint (none) -> Package_DIP:DIP-8_W7.62mm
Connections:
- net GND: now also C1.2, C2.2, J3.6 (Pin_6), J5.2 (Pin_2), J6.4 (Pin_4), R11.2, R5.2, U3.22 (GND), U3.8 (GND); no longer R9.2
- net VDD: now also C2.1, J3.2 (Pin_2), J5.1 (Pin_1), J6.1 (Pin_1), R2.2, U3.20 (AVCC), U3.7 (VCC)
- net at J2.1 (Pin_1), U1.7: now also R6.1, U3.24 (PC1); no longer R10.1
- net at J1.1 (Pin_1), R1.1, R3.1: now also C1.1, U3.15 (PB1), U3.21 (AREF)
- net at R3.2, R4.1, U2.3 (+): now also R5.1
- new net: J6.2 (Pin_2), U3.27 (PC4)
- new net: J6.3 (Pin_3), U3.28 (PC5)
- new net: J3.5 (Pin_5), R2.1, U3.1 (~{RESET}/PC6)
- new net: J3.4 (Pin_4), U3.17 (PB3)
- new net: J3.1 (Pin_1), U3.18 (PB4)
- new net: J3.3 (Pin_3), U3.19 (PB5)
- new net: R10.1, R6.2
- new net: R11.1, R9.2
Other:
- moved on the sheet: J1, J2, R1, R10, R3, R4, R7, R8, R9, Rm1, U1B, U1C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
